Commit message: Add Gazebo ros2_control and joint trajectory control

File: src/my_first_ros2_package/urdf/palletizing_robot.urdf (robot description, URDF)
Before this commit: robot palletizing_robot, 5 links, 4 joints
Links:
- added link world
- link arm_link: mass None -> 5.0; geometry collision box size=0.1 0.1 0.8; visual box size=0.1 0.1 0.8
- link base_link: mass None -> 20.0; geometry collision cylinder length=0.1 radius=0.3; visual cylinder length=0.1 radius=0.3
- link conveyor_link: mass None -> 15.0; geometry collision box size=0.4 1.5 0.05; visual box size=0.4 1.5 0.05
- link gripper_link: mass None -> 1.0; geometry collision box size=0.2 0.2 0.05; visual box size=0.2 0.2 0.05
- link torso_link: mass None -> 10.0; geometry collision cylinder length=0.5 radius=0.15; visual cylinder length=0.5 radius=0.15
Joints:
- added joint world_to_base: type fixed, parent world, child base_link, origin xyz=0 0 0.05 rpy=0 0 0

Commit message: Stabilize Gazebo ros2_control palletizing workflow

File: src/my_first_ros2_package/urdf/palletizing_robot.urdf (robot description, URDF)
Before this commit: robot palletizing_robot, 6 links, 5 joints
Joints:
- joint torso_to_arm: limit lower=-1.57 upper=1.57 effort=10.0 velocity=1.0 -> lower=-1.57 upper=1.57 effort=50.0 velocity=1.0
